File: kicad_cool640/cool640.kicad_pcb (KiCad board)
At the start: 2 copper layers, 236 x 223.2 mm, 49 parts, among them J1 MJ-4PP-9, J2 LED, SW1 SW_PUSH, SW10 SW_PUSH, SW11 SW_PUSH, SW12 SW_PUSH, SW13 SW_PUSH, SW14 SW_PUSH, SW15 SW_PUSH, SW16 SW_PUSH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

Commit message: fix
Parts:
- added J3: LED, kbd:StripLED_1side, B.Cu at (65.6, -23.1)
Routing:
- net LED: track 66.2 -> 93.2 mm, vias 5 -> 6
- net VCC: track 109.3 -> 125.1 mm, vias 0 -> 1
- net GND: track 225.7 -> 229.9 mm, vias 3 -> 5
- net data: track 101.6 -> 104.2 mm
Other:
- board text added: "Col0"
- board text added: "Col1"
- board text added: "Col2"
- board text added: "Col3"
- board text added: "Col4"
- board text added: "Row0"
- board text added: "Row1"
- board text added: "Row2"
- board text added: "Row3"
- board text added: "cool640 designed by m.ki date 20220223 ver.1.1"
- board text removed: "cool640 designed by m.ki date 20220223 ver.1.0"
