File: kicad_cool640/cool640pcbv110.kicad_pcb (KiCad board)
At the start: 2 copper layers, 236 x 223.2 mm, 50 parts, among them J1 MJ-4PP-9, J2 LED, J3 LED, SW1 SW_PUSH, SW10 SW_PUSH, SW11 SW_PUSH, SW12 SW_PUSH, SW13 SW_PUSH, SW14 SW_PUSH, SW15 SW_PUSH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

Commit message: fix
Other:
- board size 236 x 223.2 mm -> 98.2 x 99.5 mm
Changed lines of the file:
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@@
   (general
     (thickness 1.6)
-    (drawings 241)
+    (drawings 127)
     (tracks 825)
     (zones 0)
@@
       (net 31 GND))
   )
-  (gr_line (start 168.84 47.43) (end 182.84 47.43) (layer Edge.Cuts) (width 0.15))
-  (gr_line (start 168.83 52.49) (end 168.83 66.49) (layer Edge.Cuts) (width 0.15))
-  (gr_line (start 187.88 52.49) (end 187.88 66.49) (layer Edge.Cuts) (width 0.15))
-  (gr_line (start 187.89 9.33) (end 201.89 9.33) (layer Edge.Cuts) (width 0.15))
-  (gr_circle (center 204.51 171.42) (end 205.61 171.42) (layer Edge.Cuts) (width 0.15))
-  (gr_arc (start 127.38 188.76) (end 126.26 188.76) (angle -90) (layer Edge.Cuts) (width 0.15))
-  (gr_line (start 224.5 91.53) (end 224.5 110.61) (layer Edge.Cuts) (width 0.15))
-  (gr_circle (center 146.28 171.42) (end 147.38 171.42) (layer Edge.Cuts) (width 0.15))
-  (gr_line (start 127.38 189.88) (end 223.38 189.88) (layer Edge.Cuts) (width 0.15))
-  (gr_line (start 126.26 97.04) (end 126.26 188.76) (layer Edge.Cuts) (width 0.15))
-  (gr_line (start 223.38 90.41) (end 127.38 90.41) (layer Edge.Cuts) (width 0.15))
-  (gr_line (start 224.5 188.76) (end 224.5 110.61) (layer Edge.Cuts) (width 0.15))
-  (gr_circle (center 146.28 133.32) (end 147.38 133.32) (layer Edge.Cuts) (width 0.15))
-  (gr_arc (start 223.38 188.76) (end 223.38 189.88) (angle -90) (layer Edge.Cuts) (width 0.15))
-  (gr_line (start 126.26 91.53) (end 126.26 97.04) (layer Edge.Cuts) (width 0.15))
-  (gr_circle (center 204.51 133.32) (end 205.61 133.32) (layer Edge.Cuts) (width 0.15))
-  (gr_arc (start 127.77 67.32) (end 126.65 67.32) (angle -90) (layer Edge.Cuts) (width 0.15))
-  (gr_arc (start 223.77 67.32) (end 223.77 68.44) (angle -90) (layer Edge.Cuts) (width 0.15))
-  (gr_arc (start 223.77 -29.91) (end 224.89 -29.91) (angle -90) (layer Edge.Cuts) (width 0.15))
-  (gr_arc (start 127.77 -29.91) (end 127.77 -31.03) (angle -90) (layer Edge.Cuts) (width 0.15))
-  (gr_line (start 127.77 -7.62) (end 223.77 -7.62) (layer Edge.Cuts) (width 0.15))
-  (gr_line (start 126.65 -29.91) (end 126.65 -8.74) (layer Edge.Cuts) (width 0.15))
-  (gr_line (start 163.78 33.43) (end 149.78 33.43) (layer Edge.Cuts) (width 0.15))
-  (gr_line (start 149.77 14.39) (end 149.77 28.39) (layer Edge.Cuts) (width 0.15))
-  (gr_line (start 149.78 33.43) (end 149.78 47.43) (layer Edge.Cuts) (width 0.15))
-  (gr_line (start 149.78 47.43) (end 163.78 47.43) (layer Edge.Cuts) (width 0.15))
-  (gr_line (start 130.73 14.39) (end 130.73 28.39) (layer Edge.Cuts) (width 0.15))
-  (gr_line (start 130.74 33.43) (end 130.74 47.43) (layer Edge.Cuts) (width 0.15))
-  (gr_line (start 130.74 47.43) (end 144.74 47.43) (layer Edge.Cuts) (width 0.15))
-  (gr_circle (center 146.67 11.88) (end 147.77 11.88) (layer Edge.Cuts) (width 0.15))
-  (gr_line (start 168.84 9.33) (end 182.84 9.33) (layer Edge.Cuts) (width 0.15))
-  (gr_line (start 187.89 47.43) (end 201.89 47.43) (layer Edge.Cuts) (width 0.15))
-  (gr_line (start 206.93 52.49) (end 206.93 66.49) (layer Edge.Cuts) (width 0.15))
-  (gr_line (start 206.94 9.33) (end 220.94 9.33) (layer Edge.Cuts) (width 0.15))
-  (gr_line (start 206.93 66.49) (end 220.93 66.49) (layer Edge.Cuts) (width 0.15))
-  (gr_line (start 220.94 47.43) (end 220.94 33.43) (layer Edge.Cuts) (width 0.15))
-  (gr_line (start 220.93 66.49) (end 220.93 52.49) (layer Edge.Cuts) (width 0.15))
-  (gr_line (start 201.88 52.49) (end 187.88 52.49) (layer Edge.Cuts) (width 0.15))
-  (gr_circle (center 204.9 11.88) (end 206 11.88) (layer Edge.Cuts) (width 0.15))
-  (gr_line (start 163.78 47.43) (end 163.78 33.43) (layer Edge.Cuts) (width 0.15))
-  (gr_line (start 163.77 66.49) (end 163.77 52.49) (layer Edge.Cuts) (width 0.15))
-  (gr_line (start 149.77 28.39) (end 163.77 28.39) (layer Edge.Cuts) (width 0.15))
-  (gr_line (start 149.78 -4.67) (end 149.78 9.33) (layer Edge.Cuts) (width 0.15))
-  (gr_line (start 163.77 14.39) (end 149.77 14.39) (layer Edge.Cuts) (width 0.15))
-  (gr_line (start 163.77 28.39) (end 163.77 14.39) (layer Edge.Cuts) (width 0.15))
-  (gr_line (start 220.94 33.43) (end 206.94 33.43) (layer Edge.Cuts) (width 0.15))
-  (gr_line (start 220.93 28.39) (end 220.93 14.39) (layer Edge.Cuts) (width 0.15))
-  (gr_line (start 182.84 33.43) (end 168.84 33.43) (layer Edge.Cuts) (width 0.15))
-  (gr_line (start 144.74 9.33) (end 144.74 -4.67) (layer Edge.Cuts) (width 0.15))
-  (gr_line (start 130.73 66.49) (end 144.73 66.49) (layer Edge.Cuts) (width 0.15))
-  (gr_line (start 144.74 47.43) (end 144.74 33.43) (layer Edge.Cuts) (width 0.15))
-  (gr_line (start 220.93 14.39) (end 206.93 14.39) (layer Edge.Cuts) (width 0.15))
-  (gr_line (start 220.94 -4.67) (end 206.94 -4.67) (layer Edge.Cuts) (width 0.15))
-  (gr_line (start 220.94 9.33) (end 220.94 -4.67) (layer Edge.Cuts) (width 0.15))
-  (gr_line (start 127.77 68.44) (end 223.77 68.44) (layer Edge.Cuts) (width 0.15))
-  (gr_line (start 126.65 -6.74) (end 126.65 67.32) (layer Edge.Cuts) (width 0.15))
-  (gr_line (start 223.77 -31.03) (end 127.77 -31.03) (layer Edge.Cuts) (width 0.15))
-  (gr_line (start 224.89 67.32) (end 224.89 -6.74) (layer Edge.Cuts) (width 0.15))
-  (gr_line (start 130.74 -4.67) (end 130.74 9.33) (layer Edge.Cuts) (width 0.15))
-  (gr_line (start 206.93 28.39) (end 220.93 28.39) (layer Edge.Cuts) (width 0.15))
-  (gr_line (start 206.94 -4.67) (end 206.94 9.33) (layer Edge.Cuts) (width 0.15))
-  (gr_line (start 168.83 14.39) (end 168.83 28.39) (layer Edge.Cuts) (width 0.15))
-  (gr_line (start 201.88 66.49) (end 201.88 52.49) (layer Edge.Cuts) (width 0.15))
-  (gr_line (start 187.88 28.39) (end 201.88 28.39) (layer Edge.Cuts) (width 0.15))
-  (gr_line (start 187.89 -4.67) (end 187.89 9.33) (layer Edge.Cuts) (width 0.15))
-  (gr_line (start 201.88 14.39) (end 187.88 14.39) (layer Edge.Cuts) (width 0.15))
-  (gr_line (start 201.89 -4.67) (end 187.89 -4.67) (layer Edge.Cuts) (width 0.15))
-  (gr_line (start 201.89 9.33) (end 201.89 -4.67) (layer Edge.Cuts) (width 0.15))
-  (gr_line (start 187.88 14.39) (end 187.88 28.39) (layer Edge.Cuts) (width 0.15))
-  (gr_line (start 187.89 33.43) (end 187.89 47.43) (layer Edge.Cuts) (width 0.15))
-  (gr_line (start 168.83 66.49) (end 182.83 66.49) (layer Edge.Cuts) (width 0.15))
-  (gr_line (start 182.84 47.43) (end 182.84 33.43) (layer Edge.Cuts) (width 0.15))
-  (gr_line (start 182.83 66.49) (end 182.83 52.49) (layer Edge.Cuts) (width 0.15))
-  (gr_line (start 168.83 28.39) (end 182.83 28.39) (layer Edge.Cuts) (width 0.15))
-  (gr_line (start 168.84 -4.67) (end 168.84 9.33) (layer Edge.Cuts) (width 0.15))
-  (gr_line (start 182.83 14.39) (end 168.83 14.39) (layer Edge.Cuts) (width 0.15))
-  (gr_line (start 182.83 28.39) (end 182.83 14.39) (layer Edge.Cuts) (width 0.15))
-  (gr_line (start 144.74 33.43) (end 130.74 33.43) (layer Edge.Cuts) (width 0.15))
-  (gr_line (start 149.77 52.49) (end 149.77 66.49) (layer Edge.Cuts) (width 0.15))
-  (gr_line (start 149.78 9.33) (end 163.78 9.33) (layer Edge.Cuts) (width 0.15))
-  (gr_line (start 187.88 66.49) (end 201.88 66.49) (layer Edge.Cuts) (width 0.15))
-  (gr_line (start 201.89 47.43) (end 201.89 33.43) (layer Edge.Cuts) (width 0.15))
-  (gr_line (start 182.84 9.33) (end 182.84 -4.67) (layer Edge.Cuts) (width 0.15))
-  (gr_line (start 206.93 14.39) (end 206.93 28.39) (layer Edge.Cuts) (width 0.15))
-  (gr_line (start 206.94 33.43) (end 206.94 47.43) (layer Edge.Cuts) (width 0.15))
-  (gr_line (start 220.93 52.49) (end 206.93 52.49) (layer Edge.Cuts) (width 0.15))
-  (gr_line (start 206.94 47.43) (end 220.94 47.43) (layer Edge.Cuts) (width 0.15))
-  (gr_line (start 144.73 66.49) (end 144.73 52.49) (layer Edge.Cuts) (width 0.15))
-  (gr_line (start 144.73 52.49) (end 130.73 52.49) (layer Edge.Cuts) (width 0.15))
-  (gr_line (start 163.77 52.49) (end 149.77 52.49) (layer Edge.Cuts) (width 0.15))
-  (gr_line (start 163.78 -4.67) (end 149.78 -4.67) (layer Edge.Cuts) (width 0.15))
-  (gr_line (start 163.78 9.33) (end 163.78 -4.67) (layer Edge.Cuts) (width 0.15))
-  (gr_line (start 149.77 66.49) (end 163.77 66.49) (layer Edge.Cuts) (width 0.15))
-  (gr_line (start 224.89 -6.74) (end 126.65 -6.74) (layer Edge.Cuts) (width 0.15))
-  (gr_circle (center 146.67 49.98) (end 147.77 49.98) (layer Edge.Cuts) (width 0.15))
-  (gr_line (start 144.74 -4.67) (end 130.74 -4.67) (layer Edge.Cuts) (width 0.15))
-  (gr_circle (center 204.9 49.98) (end 206 49.98) (layer Edge.Cuts) (width 0.15))
-  (gr_line (start 130.73 52.49) (end 130.73 66.49) (layer Edge.Cuts) (width 0.15))
-  (gr_line (start 130.74 9.33) (end 144.74 9.33) (layer Edge.Cuts) (width 0.15))
-  (gr_circle (center 134.44 -18.02) (end 135.54 -18.02) (layer Edge.Cuts) (width 0.15))
-  (gr_line (start 144.73 14.39) (end 130.73 14.39) (layer Edge.Cuts) (width 0.15))
-  (gr_line (start 144.73 28.39) (end 144.73 14.39) (layer Edge.Cuts) (width 0.15))
-  (gr_line (start 130.73 28.39) (end 144.73 28.39) (layer Edge.Cuts) (width 0.15))
-  (gr_line (start 224.89 -29.91) (end 224.89 -8.74) (layer Edge.Cuts) (width 0.15))
-  (gr_arc (start 223.38 91.53) (end 224.5 91.53) (angle -90) (layer Edge.Cuts) (width 0.15))
-  (gr_arc (start 127.38 91.53) (end 127.38 90.41) (angle -90) (layer Edge.Cuts) (width 0.15))
-  (gr_circle (center 151.12 -17.92) (end 152.22 -17.92) (layer Edge.Cuts) (width 0.15))
-  (gr_arc (start 127.77 -8.74) (end 126.65 -8.74) (angle -90) (layer Edge.Cuts) (width 0.15))
-  (gr_arc (start 223.77 -8.74) (end 223.77 -7.62) (angle -90) (layer Edge.Cuts) (width 0.15))
-  (gr_line (start 201.89 33.43) (end 187.89 33.43) (layer Edge.Cuts) (width 0.15))
-  (gr_line (start 168.84 33.43) (end 168.84 47.43) (layer Edge.Cuts) (width 0.15))
-  (gr_line (start 182.84 -4.67) (end 168.84 -4.67) (layer Edge.Cuts) (width 0.15))
-  (gr_line (start 201.88 28.39) (end 201.88 14.39) (layer Edge.Cuts) (width 0.15))
-  (gr_line (start 182.83 52.49) (end 168.83 52.49) (layer Edge.Cuts) (width 0.15))
   (gr_text Row0 (at -9.45 -1.1 90) (layer F.SilkS)
     (effects (font (size 1.5 1.5) (thickness 0.3)))
