File: kicad_cool640/cool640.sch (KiCad schematic (older format))
At the start: 45 parts, among them J1 MJ-4PP-9, J2 LED, SW1 SW_PUSH, SW10 SW_PUSH, SW11 SW_PUSH, SW12 SW_PUSH, SW13 SW_PUSH, SW14 SW_PUSH, SW15 SW_PUSH, SW16 SW_PUSH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

Commit message: fix
Parts:
- added J3: LED, kbd:StripLED_1side, symbol Connector_Generic:Conn_01x03
- U1: symbol kbd:ProMicro -> cool640-rescue:ProMicro-kbd
- U2: symbol Pico:PICO_RP2040 -> cool640-rescue:PICO_RP2040-Pico
Connections:
- net GND: now also J3.1 (Pin_1)
- net LED: now also J3.2 (Pin_2)
- net VCC: now also J3.3 (Pin_3)
Changed lines of the file:
@@
 $EndDescr
 $Comp
-L kbd:ProMicro U1
+L cool640-rescue:ProMicro-kbd U1
 U 1 1 61F92BBE
 P 3600 1925
@@
 $EndComp
 $Comp
-L Pico:PICO_RP2040 U2
+L cool640-rescue:PICO_RP2040-Pico U2
 U 1 1 621738D9
 P 7675 2200
@@
 Wire Wire Line
 	5125 2825 5125 3125
+$Comp
+L Connector_Generic:Conn_01x03 J3
+U 1 1 622800E0
+P 950 3125
+F 0 "J3" H 868 2800 50  0000 C CNN
+F 1 "LED" H 868 2891 50  0000 C CNN
+F 2 "kbd:StripLED_1side" H 950 3125 50  0001 C CNN
+F 3 "~" H 950 3125 50  0001 C CNN
+	1    950  3125
+	-1   0    0    1
+$EndComp
+Text GLabel 1150 3125 2    50   Input ~ 0
+LED
+$Comp
+L power:VCC #PWR0114
+U 1 1 622800EB
+P 1375 3025
+F 0 "#PWR0114" H 1375 2875 50  0001 C CNN
+F 1 "VCC" H 1390 3198 50  0000 C CNN
+F 2 "" H 1375 3025 50  0001 C CNN
+F 3 "" H 1375 3025 50  0001 C CNN
+	1    1375 3025
+	1    0    0    -1
+$EndComp
+$Comp
+L power:GND #PWR0115
+U 1 1 622800F5
+P 1375 3225
+F 0 "#PWR0115" H 1375 2975 50  0001 C CNN
+F 1 "GND" H 1380 3052 50  0000 C CNN
+F 2 "" H 1375 3225 50  0001 C CNN
+F 3 "" H 1375 3225 50  0001 C CNN
+	1    1375 3225
+	1    0    0    -1
+$EndComp
+Wire Wire Line
+	1150 3225 1375 3225
+Wire Wire Line
+	1150 3025 1375 3025
 $EndSCHEMATC

Commit message: fix
Parts:
- SW1, SW10, SW11, SW12, SW13, SW14, SW15, SW16, SW17, SW18, SW19, SW2, SW20, SW3, SW4, SW5, SW6, SW7, SW8, SW9: footprint kbd:CherryMX_MidHeight_Choc_Hotswap_katagawa -> logo:CherryMX_MidHeight_Choc_Hotswap_katagawa
Changed lines of the file:
@@
 F 0 "SW1" H 2150 3380 50  0000 C CNN
 F 1 "SW_PUSH" H 2150 3289 50  0000 C CNN
-F 2 "kbd:CherryMX_MidHeight_Choc_Hotswap_katagawa" H 2150 3125 50  0001 C CNN
+F 2 "logo:CherryMX_MidHeight_Choc_Hotswap_katagawa" H 2150 3125 50  0001 C CNN
 F 3 "" H 2150 3125 50  0000 C CNN
 	1    2150 3125
@@
 F 0 "SW2" H 2975 3380 50  0000 C CNN
 F 1 "SW_PUSH" H 2975 3289 50  0000 C CNN
-F 2 "kbd:CherryMX_MidHeight_Choc_Hotswap_katagawa" H 2975 3125 50  0001 C CNN
+F 2 "logo:CherryMX_MidHeight_Choc_Hotswap_katagawa" H 2975 3125 50  0001 C CNN
 F 3 "" H 2975 3125 50  0000 C CNN
 	1    2975 3125
@@
 F 0 "SW3" H 3775 3380 50  0000 C CNN
 F 1 "SW_PUSH" H 3775 3289 50  0000 C CNN
-F 2 "kbd:CherryMX_MidHeight_Choc_Hotswap_katagawa" H 3775 3125 50  0001 C CNN
+F 2 "logo:CherryMX_MidHeight_Choc_Hotswap_katagawa" H 3775 3125 50  0001 C CNN
 F 3 "" H 3775 3125 50  0000 C CNN
 	1    3775 3125
@@
 F 0 "SW4" H 4600 3380 50  0000 C CNN
 F 1 "SW_PUSH" H 4600 3289 50  0000 C CNN
-F 2 "kbd:CherryMX_MidHeight_Choc_Hotswap_katagawa" H 4600 3125 50  0001 C CNN
+F 2 "logo:CherryMX_MidHeight_Choc_Hotswap_katagawa" H 4600 3125 50  0001 C CNN
 F 3 "" H 4600 3125 50  0000 C CNN
 	1    4600 3125
@@
 F 0 "SW6" H 2150 4130 50  0000 C CNN
 F 1 "SW_PUSH" H 2150 4039 50  0000 C CNN
-F 2 "kbd:CherryMX_MidHeight_Choc_Hotswap_katagawa" H 2150 3875 50  0001 C CNN
+F 2 "logo:CherryMX_MidHeight_Choc_Hotswap_katagawa" H 2150 3875 50  0001 C CNN
 F 3 "" H 2150 3875 50  0000 C CNN
 	1    2150 3875
@@
 F 0 "SW7" H 2975 4130 50  0000 C CNN
 F 1 "SW_PUSH" H 2975 4039 50  0000 C CNN
-F 2 "kbd:CherryMX_MidHeight_Choc_Hotswap_katagawa" H 2975 3875 50  0001 C CNN
+F 2 "logo:CherryMX_MidHeight_Choc_Hotswap_katagawa" H 2975 3875 50  0001 C CNN
 F 3 "" H 2975 3875 50  0000 C CNN
 	1    2975 3875
@@
 F 0 "SW8" H 3775 4130 50  0000 C CNN
 F 1 "SW_PUSH" H 3775 4039 50  0000 C CNN
-F 2 "kbd:CherryMX_MidHeight_Choc_Hotswap_katagawa" H 3775 3875 50  0001 C CNN
+F 2 "logo:CherryMX_MidHeight_Choc_Hotswap_katagawa" H 3775 3875 50  0001 C CNN
 F 3 "" H 3775 3875 50  0000 C CNN
 	1    3775 3875
@@
 F 0 "SW9" H 4600 4130 50  0000 C CNN
 F 1 "SW_PUSH" H 4600 4039 50  0000 C CNN
-F 2 "kbd:CherryMX_MidHeight_Choc_Hotswap_katagawa" H 4600 3875 50  0001 C CNN
+F 2 "logo:CherryMX_MidHeight_Choc_Hotswap_katagawa" H 4600 3875 50  0001 C CNN
 F 3 "" H 4600 3875 50  0000 C CNN
 	1    4600 3875
@@
 F 0 "SW11" H 2150 4880 50  0000 C CNN
 F 1 "SW_PUSH" H 2150 4789 50  0000 C CNN
-F 2 "kbd:CherryMX_MidHeight_Choc_Hotswap_katagawa" H 2150 4625 50  0001 C CNN
+F 2 "logo:CherryMX_MidHeight_Choc_Hotswap_katagawa" H 2150 4625 50  0001 C CNN
 F 3 "" H 2150 4625 50  0000 C CNN
 	1    2150 4625
@@
 F 0 "SW12" H 2975 4880 50  0000 C CNN
 F 1 "SW_PUSH" H 2975 4789 50  0000 C CNN
-F 2 "kbd:CherryMX_MidHeight_Choc_Hotswap_katagawa" H 2975 4625 50  0001 C CNN
+F 2 "logo:CherryMX_MidHeight_Choc_Hotswap_katagawa" H 2975 4625 50  0001 C CNN
 F 3 "" H 2975 4625 50  0000 C CNN
 	1    2975 4625
@@
 F 0 "SW13" H 3775 4880 50  0000 C CNN
 F 1 "SW_PUSH" H 3775 4789 50  0000 C CNN
-F 2 "kbd:CherryMX_MidHeight_Choc_Hotswap_katagawa" H 3775 4625 50  0001 C CNN
+F 2 "logo:CherryMX_MidHeight_Choc_Hotswap_katagawa" H 3775 4625 50  0001 C CNN
 F 3 "" H 3775 4625 50  0000 C CNN
 	1    3775 4625
@@
 F 0 "SW14" H 4600 4880 50  0000 C CNN
 F 1 "SW_PUSH" H 4600 4789 50  0000 C CNN
-F 2 "kbd:CherryMX_MidHeight_Choc_Hotswap_katagawa" H 4600 4625 50  0001 C CNN
+F 2 "logo:CherryMX_MidHeight_Choc_Hotswap_katagawa" H 4600 4625 50  0001 C CNN
 F 3 "" H 4600 4625 50  0000 C CNN
 	1    4600 4625
@@
 F 0 "SW16" H 2150 5630 50  0000 C CNN
 F 1 "SW_PUSH" H 2150 5539 50  0000 C CNN
-F 2 "kbd:CherryMX_MidHeight_Choc_Hotswap_katagawa" H 2150 5375 50  0001 C CNN
+F 2 "logo:CherryMX_MidHeight_Choc_Hotswap_katagawa" H 2150 5375 50  0001 C CNN
 F 3 "" H 2150 5375 50  0000 C CNN
 	1    2150 5375
@@
 F 0 "SW17" H 2975 5630 50  0000 C CNN
 F 1 "SW_PUSH" H 2975 5539 50  0000 C CNN
-F 2 "kbd:CherryMX_MidHeight_Choc_Hotswap_katagawa" H 2975 5375 50  0001 C CNN
+F 2 "logo:CherryMX_MidHeight_Choc_Hotswap_katagawa" H 2975 5375 50  0001 C CNN
 F 3 "" H 2975 5375 50  0000 C CNN
 	1    2975 5375
@@
 F 0 "SW18" H 3775 5630 50  0000 C CNN
 F 1 "SW_PUSH" H 3775 5539 50  0000 C CNN
-F 2 "kbd:CherryMX_MidHeight_Choc_Hotswap_katagawa" H 3775 5375 50  0001 C CNN
+F 2 "logo:CherryMX_MidHeight_Choc_Hotswap_katagawa" H 3775 5375 50  0001 C CNN
 F 3 "" H 3775 5375 50  0000 C CNN
 	1    3775 5375
@@
 F 0 "SW19" H 4600 5630 50  0000 C CNN
 F 1 "SW_PUSH" H 4600 5539 50  0000 C CNN
-F 2 "kbd:CherryMX_MidHeight_Choc_Hotswap_katagawa" H 4600 5375 50  0001 C CNN
+F 2 "logo:CherryMX_MidHeight_Choc_Hotswap_katagawa" H 4600 5375 50  0001 C CNN
 F 3 "" H 4600 5375 50  0000 C CNN
 	1    4600 5375
@@
 F 0 "SW5" H 5425 3380 50  0000 C CNN
 F 1 "SW_PUSH" H 5425 3289 50  0000 C CNN
-F 2 "kbd:CherryMX_MidHeight_Choc_Hotswap_katagawa" H 5425 3125 50  0001 C CNN
+F 2 "logo:CherryMX_MidHeight_Choc_Hotswap_katagawa" H 5425 3125 50  0001 C CNN
 F 3 "" H 5425 3125 50  0000 C CNN
 	1    5425 3125
@@
 F 0 "SW10" H 5425 4130 50  0000 C CNN
 F 1 "SW_PUSH" H 5425 4039 50  0000 C CNN
-F 2 "kbd:CherryMX_MidHeight_Choc_Hotswap_katagawa" H 5425 3875 50  0001 C CNN
+F 2 "logo:CherryMX_MidHeight_Choc_Hotswap_katagawa" H 5425 3875 50  0001 C CNN
 F 3 "" H 5425 3875 50  0000 C CNN
 	1    5425 3875
@@
 F 0 "SW15" H 5425 4880 50  0000 C CNN
 F 1 "SW_PUSH" H 5425 4789 50  0000 C CNN
-F 2 "kbd:CherryMX_MidHeight_Choc_Hotswap_katagawa" H 5425 4625 50  0001 C CNN
+F 2 "logo:CherryMX_MidHeight_Choc_Hotswap_katagawa" H 5425 4625 50  0001 C CNN
 F 3 "" H 5425 4625 50  0000 C CNN
 	1    5425 4625
@@
 F 0 "SW20" H 5425 5630 50  0000 C CNN
 F 1 "SW_PUSH" H 5425 5539 50  0000 C CNN
-F 2 "kbd:CherryMX_MidHeight_Choc_Hotswap_katagawa" H 5425 5375 50  0001 C CNN
+F 2 "logo:CherryMX_MidHeight_Choc_Hotswap_katagawa" H 5425 5375 50  0001 C CNN
 F 3 "" H 5425 5375 50  0000 C CNN
 	1    5425 5375
