File: kicad_cool640/cool640pcbv110.sch (KiCad schematic (older format))
At the start: 46 parts, among them J1 MJ-4PP-9, J2 LED, J3 LED, SW1 SW_PUSH, SW10 SW_PUSH, SW11 SW_PUSH, SW12 SW_PUSH, SW13 SW_PUSH, SW14 SW_PUSH, SW15 SW_PUSH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

Commit message: fix
Parts:
- SW1, SW10, SW11, SW12, SW13, SW14, SW15, SW16, SW17, SW18, SW19, SW2, SW20, SW3, SW4, SW5, SW6, SW7, SW8, SW9: footprint kbd:CherryMX_MidHeight_Choc_Hotswap -> kbd:CherryMX_MidHeight_Choc_Hotswap_katagawa
Changed lines of the file:
@@
 F 0 "SW1" H 2150 3380 50  0000 C CNN
 F 1 "SW_PUSH" H 2150 3289 50  0000 C CNN
-F 2 "kbd:CherryMX_MidHeight_Choc_Hotswap" H 2150 3125 50  0001 C CNN
+F 2 "kbd:CherryMX_MidHeight_Choc_Hotswap_katagawa" H 2150 3125 50  0001 C CNN
 F 3 "" H 2150 3125 50  0000 C CNN
 	1    2150 3125
@@
 F 0 "SW2" H 2975 3380 50  0000 C CNN
 F 1 "SW_PUSH" H 2975 3289 50  0000 C CNN
-F 2 "kbd:CherryMX_MidHeight_Choc_Hotswap" H 2975 3125 50  0001 C CNN
+F 2 "kbd:CherryMX_MidHeight_Choc_Hotswap_katagawa" H 2975 3125 50  0001 C CNN
 F 3 "" H 2975 3125 50  0000 C CNN
 	1    2975 3125
@@
 F 0 "SW3" H 3775 3380 50  0000 C CNN
 F 1 "SW_PUSH" H 3775 3289 50  0000 C CNN
-F 2 "kbd:CherryMX_MidHeight_Choc_Hotswap" H 3775 3125 50  0001 C CNN
+F 2 "kbd:CherryMX_MidHeight_Choc_Hotswap_katagawa" H 3775 3125 50  0001 C CNN
 F 3 "" H 3775 3125 50  0000 C CNN
 	1    3775 3125
@@
 F 0 "SW4" H 4600 3380 50  0000 C CNN
 F 1 "SW_PUSH" H 4600 3289 50  0000 C CNN
-F 2 "kbd:CherryMX_MidHeight_Choc_Hotswap" H 4600 3125 50  0001 C CNN
+F 2 "kbd:CherryMX_MidHeight_Choc_Hotswap_katagawa" H 4600 3125 50  0001 C CNN
 F 3 "" H 4600 3125 50  0000 C CNN
 	1    4600 3125
@@
 F 0 "SW6" H 2150 4130 50  0000 C CNN
 F 1 "SW_PUSH" H 2150 4039 50  0000 C CNN
-F 2 "kbd:CherryMX_MidHeight_Choc_Hotswap" H 2150 3875 50  0001 C CNN
+F 2 "kbd:CherryMX_MidHeight_Choc_Hotswap_katagawa" H 2150 3875 50  0001 C CNN
 F 3 "" H 2150 3875 50  0000 C CNN
 	1    2150 3875
@@
 F 0 "SW7" H 2975 4130 50  0000 C CNN
 F 1 "SW_PUSH" H 2975 4039 50  0000 C CNN
-F 2 "kbd:CherryMX_MidHeight_Choc_Hotswap" H 2975 3875 50  0001 C CNN
+F 2 "kbd:CherryMX_MidHeight_Choc_Hotswap_katagawa" H 2975 3875 50  0001 C CNN
 F 3 "" H 2975 3875 50  0000 C CNN
 	1    2975 3875
@@
 F 0 "SW8" H 3775 4130 50  0000 C CNN
 F 1 "SW_PUSH" H 3775 4039 50  0000 C CNN
-F 2 "kbd:CherryMX_MidHeight_Choc_Hotswap" H 3775 3875 50  0001 C CNN
+F 2 "kbd:CherryMX_MidHeight_Choc_Hotswap_katagawa" H 3775 3875 50  0001 C CNN
 F 3 "" H 3775 3875 50  0000 C CNN
 	1    3775 3875
@@
 F 0 "SW9" H 4600 4130 50  0000 C CNN
 F 1 "SW_PUSH" H 4600 4039 50  0000 C CNN
-F 2 "kbd:CherryMX_MidHeight_Choc_Hotswap" H 4600 3875 50  0001 C CNN
+F 2 "kbd:CherryMX_MidHeight_Choc_Hotswap_katagawa" H 4600 3875 50  0001 C CNN
 F 3 "" H 4600 3875 50  0000 C CNN
 	1    4600 3875
@@
 F 0 "SW11" H 2150 4880 50  0000 C CNN
 F 1 "SW_PUSH" H 2150 4789 50  0000 C CNN
-F 2 "kbd:CherryMX_MidHeight_Choc_Hotswap" H 2150 4625 50  0001 C CNN
+F 2 "kbd:CherryMX_MidHeight_Choc_Hotswap_katagawa" H 2150 4625 50  0001 C CNN
 F 3 "" H 2150 4625 50  0000 C CNN
 	1    2150 4625
@@
 F 0 "SW12" H 2975 4880 50  0000 C CNN
 F 1 "SW_PUSH" H 2975 4789 50  0000 C CNN
-F 2 "kbd:CherryMX_MidHeight_Choc_Hotswap" H 2975 4625 50  0001 C CNN
+F 2 "kbd:CherryMX_MidHeight_Choc_Hotswap_katagawa" H 2975 4625 50  0001 C CNN
 F 3 "" H 2975 4625 50  0000 C CNN
 	1    2975 4625
@@
 F 0 "SW13" H 3775 4880 50  0000 C CNN
 F 1 "SW_PUSH" H 3775 4789 50  0000 C CNN
-F 2 "kbd:CherryMX_MidHeight_Choc_Hotswap" H 3775 4625 50  0001 C CNN
+F 2 "kbd:CherryMX_MidHeight_Choc_Hotswap_katagawa" H 3775 4625 50  0001 C CNN
 F 3 "" H 3775 4625 50  0000 C CNN
 	1    3775 4625
@@
 F 0 "SW14" H 4600 4880 50  0000 C CNN
 F 1 "SW_PUSH" H 4600 4789 50  0000 C CNN
-F 2 "kbd:CherryMX_MidHeight_Choc_Hotswap" H 4600 4625 50  0001 C CNN
+F 2 "kbd:CherryMX_MidHeight_Choc_Hotswap_katagawa" H 4600 4625 50  0001 C CNN
 F 3 "" H 4600 4625 50  0000 C CNN
 	1    4600 4625
@@
 F 0 "SW16" H 2150 5630 50  0000 C CNN
 F 1 "SW_PUSH" H 2150 5539 50  0000 C CNN
-F 2 "kbd:CherryMX_MidHeight_Choc_Hotswap" H 2150 5375 50  0001 C CNN
+F 2 "kbd:CherryMX_MidHeight_Choc_Hotswap_katagawa" H 2150 5375 50  0001 C CNN
 F 3 "" H 2150 5375 50  0000 C CNN
 	1    2150 5375
@@
 F 0 "SW17" H 2975 5630 50  0000 C CNN
 F 1 "SW_PUSH" H 2975 5539 50  0000 C CNN
-F 2 "kbd:CherryMX_MidHeight_Choc_Hotswap" H 2975 5375 50  0001 C CNN
+F 2 "kbd:CherryMX_MidHeight_Choc_Hotswap_katagawa" H 2975 5375 50  0001 C CNN
 F 3 "" H 2975 5375 50  0000 C CNN
 	1    2975 5375
@@
 F 0 "SW18" H 3775 5630 50  0000 C CNN
 F 1 "SW_PUSH" H 3775 5539 50  0000 C CNN
-F 2 "kbd:CherryMX_MidHeight_Choc_Hotswap" H 3775 5375 50  0001 C CNN
+F 2 "kbd:CherryMX_MidHeight_Choc_Hotswap_katagawa" H 3775 5375 50  0001 C CNN
 F 3 "" H 3775 5375 50  0000 C CNN
 	1    3775 5375
@@
 F 0 "SW19" H 4600 5630 50  0000 C CNN
 F 1 "SW_PUSH" H 4600 5539 50  0000 C CNN
-F 2 "kbd:CherryMX_MidHeight_Choc_Hotswap" H 4600 5375 50  0001 C CNN
+F 2 "kbd:CherryMX_MidHeight_Choc_Hotswap_katagawa" H 4600 5375 50  0001 C CNN
 F 3 "" H 4600 5375 50  0000 C CNN
 	1    4600 5375
@@
 F 0 "SW5" H 5425 3380 50  0000 C CNN
 F 1 "SW_PUSH" H 5425 3289 50  0000 C CNN
-F 2 "kbd:CherryMX_MidHeight_Choc_Hotswap" H 5425 3125 50  0001 C CNN
+F 2 "kbd:CherryMX_MidHeight_Choc_Hotswap_katagawa" H 5425 3125 50  0001 C CNN
 F 3 "" H 5425 3125 50  0000 C CNN
 	1    5425 3125
@@
 F 0 "SW10" H 5425 4130 50  0000 C CNN
 F 1 "SW_PUSH" H 5425 4039 50  0000 C CNN
-F 2 "kbd:CherryMX_MidHeight_Choc_Hotswap" H 5425 3875 50  0001 C CNN
+F 2 "kbd:CherryMX_MidHeight_Choc_Hotswap_katagawa" H 5425 3875 50  0001 C CNN
 F 3 "" H 5425 3875 50  0000 C CNN
 	1    5425 3875
@@
 F 0 "SW15" H 5425 4880 50  0000 C CNN
 F 1 "SW_PUSH" H 5425 4789 50  0000 C CNN
-F 2 "kbd:CherryMX_MidHeight_Choc_Hotswap" H 5425 4625 50  0001 C CNN
+F 2 "kbd:CherryMX_MidHeight_Choc_Hotswap_katagawa" H 5425 4625 50  0001 C CNN
 F 3 "" H 5425 4625 50  0000 C CNN
 	1    5425 4625
@@
 F 0 "SW20" H 5425 5630 50  0000 C CNN
 F 1 "SW_PUSH" H 5425 5539 50  0000 C CNN
-F 2 "kbd:CherryMX_MidHeight_Choc_Hotswap" H 5425 5375 50  0001 C CNN
+F 2 "kbd:CherryMX_MidHeight_Choc_Hotswap_katagawa" H 5425 5375 50  0001 C CNN
 F 3 "" H 5425 5375 50  0000 C CNN
 	1    5425 5375
