File: kicad_cool640/cool640plate_wide.kicad_pcb (KiCad board)
At the start: 2 copper layers, 499.1 x 299.2 mm, 50 parts, among them J1 MJ-4PP-9, J2 LED, J3 LED, SW1 SW_PUSH, SW10 SW_PUSH, SW11 SW_PUSH, SW12 SW_PUSH, SW13 SW_PUSH, SW14 SW_PUSH, SW15 SW_PUSH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

Commit message: fix
Parts:
- removed kiritori (x4): kiritoriparts, logo:kiritoriparts
