File: kicad_cool640/cool640x2.kicad_pcb (KiCad board)
At the start: 2 copper layers, 89.7 x 23.6 mm, 2 parts, among them U1 ProMicro, U2 PICO_RP2040

Commit message: fix
Other:
- board size 89.7 x 23.6 mm -> 283.7 x 167.7 mm
