File: kicad_cool640/cool640plate.kicad_pcb (KiCad board)
At the start: 2 copper layers, 98.6 x 220.9 mm, 0 parts

Commit message: fix
Parts:
- added D1: DIODE, kbd:D3_TH_SMD, F.Cu at (8.11, 2.36)
- added D10: DIODE, kbd:D3_TH_SMD, F.Cu at (84.2, 21.5)
- added D11: DIODE, kbd:D3_TH_SMD, F.Cu at (8.03, 40.5)
- added D12: DIODE, kbd:D3_TH_SMD, F.Cu at (27.1, 40.5)
- added D13: DIODE, kbd:D3_TH_SMD, F.Cu at (46.1, 40.5)
- added D14: DIODE, kbd:D3_TH_SMD, F.Cu at (65.2, 40.5)
- added D15: DIODE, kbd:D3_TH_SMD, F.Cu at (84.2, 40.5)
- added D16: DIODE, kbd:D3_TH_SMD, F.Cu at (8.05, 59.5)
- added D17: DIODE, kbd:D3_TH_SMD, F.Cu at (27.1, 59.5)
- added D18: DIODE, kbd:D3_TH_SMD, F.Cu at (46.2, 59.5)
- added D19: DIODE, kbd:D3_TH_SMD, F.Cu at (65.2, 59.5)
- added D2: DIODE, kbd:D3_TH_SMD, F.Cu at (27.2, 2.40)
- added D20: DIODE, kbd:D3_TH_SMD, F.Cu at (84.3, 59.6)
- added D3: DIODE, kbd:D3_TH_SMD, F.Cu at (46.1, 2.45)
- added D4: DIODE, kbd:D3_TH_SMD, F.Cu at (65.2, 2.33)
- added D5: DIODE, kbd:D3_TH_SMD, F.Cu at (84.3, 2.39)
- added D6: DIODE, kbd:D3_TH_SMD, F.Cu at (8.07, 21.4)
- added D7: DIODE, kbd:D3_TH_SMD, F.Cu at (27.1, 21.4)
- added D8: DIODE, kbd:D3_TH_SMD, F.Cu at (46.1, 21.5)
- added D9: DIODE, kbd:D3_TH_SMD, F.Cu at (65.2, 21.4)
- added J1: MJ-4PP-9, kbd:MJ-4PP-9_1side, F.Cu at (29.5, -32.0)
- added J2: LED, kbd:StripLED_1side, B.Cu at (9.62, -18.1)
- added J3: LED, kbd:StripLED_1side, B.Cu at (65.6, -23.1)
- added SW1: SW_PUSH, kbd:CherryMX_MidHeight_Choc_Hotswap_katagawa, F.Cu at (0.00, 0.00)
- added SW10: SW_PUSH, kbd:CherryMX_MidHeight_Choc_Hotswap_katagawa, F.Cu at (76.2, 19.1)
- added SW11: SW_PUSH, kbd:CherryMX_MidHeight_Choc_Hotswap_katagawa, F.Cu at (0.00, 38.1)
- added SW12: SW_PUSH, kbd:CherryMX_MidHeight_Choc_Hotswap_katagawa, F.Cu at (19.1, 38.1)
- added SW13: SW_PUSH, kbd:CherryMX_MidHeight_Choc_Hotswap_katagawa, F.Cu at (38.1, 38.1)
- added SW14: SW_PUSH, kbd:CherryMX_MidHeight_Choc_Hotswap_katagawa, F.Cu at (57.1, 38.1)
- added SW15: SW_PUSH, kbd:CherryMX_MidHeight_Choc_Hotswap_katagawa, F.Cu at (76.2, 38.1)
- added SW16: SW_PUSH, kbd:CherryMX_MidHeight_Choc_Hotswap_katagawa, F.Cu at (0.00, 57.1)
- added SW17: SW_PUSH, kbd:CherryMX_MidHeight_Choc_Hotswap_katagawa, F.Cu at (19.1, 57.1)
- added SW18: SW_PUSH, kbd:CherryMX_MidHeight_Choc_Hotswap_katagawa, F.Cu at (38.1, 57.1)
- added SW19: SW_PUSH, kbd:CherryMX_MidHeight_Choc_Hotswap_katagawa, F.Cu at (57.1, 57.1)
- added SW2: SW_PUSH, kbd:CherryMX_MidHeight_Choc_Hotswap_katagawa, F.Cu at (19.1, 0.00)
- added SW20: SW_PUSH, kbd:CherryMX_MidHeight_Choc_Hotswap_katagawa, F.Cu at (76.2, 57.1)
- added SW21: SW_PUSH, kbd:ResetSW_1side, F.Cu at (29.9, -15.6)
- added SW3: SW_PUSH, kbd:CherryMX_MidHeight_Choc_Hotswap_katagawa, F.Cu at (38.1, 0.00)
- added SW4: SW_PUSH, kbd:CherryMX_MidHeight_Choc_Hotswap_katagawa, F.Cu at (57.1, 0.00)
- added SW5: SW_PUSH, kbd:CherryMX_MidHeight_Choc_Hotswap_katagawa, F.Cu at (76.2, 0.00)
- added SW6: SW_PUSH, kbd:CherryMX_MidHeight_Choc_Hotswap_katagawa, F.Cu at (0.00, 19.1)
- added SW7: SW_PUSH, kbd:CherryMX_MidHeight_Choc_Hotswap_katagawa, F.Cu at (19.1, 19.1)
- added SW8: SW_PUSH, kbd:CherryMX_MidHeight_Choc_Hotswap_katagawa, F.Cu at (38.1, 19.1)
- added SW9: SW_PUSH, kbd:CherryMX_MidHeight_Choc_Hotswap_katagawa, F.Cu at (57.1, 19.1)
- added U1: ProMicro, logo:ProMicro_v3_kimura, F.Cu at (9.80, -20.3)
- added U2: PICO_RP2040, Pico:RPi_Pico_SMD_TH, B.Cu at (61.1, -20.8)
- added kiritori: kiritoriparts, logo:kiritoriparts, F.Cu at (81.3, -14.5)
- added kiritori: kiritoriparts, logo:kiritoriparts, F.Cu at (81.3, -27.0)
- added kiritori: kiritoriparts, logo:kiritoriparts, F.Cu at (-2.55, -15.1)
- added kiritori: kiritoriparts, logo:kiritoriparts, F.Cu at (-2.60, -25.4)
Routing:
- net row3: track 0.00 -> 365.6 mm, vias 0 -> 1
- net row2: track 0.00 -> 326.2 mm, vias 0 -> 9
- net row1: track 0.00 -> 286.9 mm, vias 0 -> 8
- net row0: track 0.00 -> 230.0 mm, vias 0 -> 8
- net GND: track 0.00 -> 229.9 mm, vias 0 -> 5
- net col4: track 0.00 -> 129.8 mm
- net col3: track 0.00 -> 129.0 mm
- net VCC: track 0.00 -> 125.1 mm, vias 0 -> 1
- net col0: track 0.00 -> 123.6 mm
- net col2: track 0.00 -> 114.0 mm, vias 0 -> 2
- net col1: track 0.00 -> 110.5 mm, vias 0 -> 2
- net data: track 0.00 -> 104.2 mm
- net LED: track 0.00 -> 93.2 mm, vias 0 -> 6
- net Net-(SW21-Pad1): track 0.00 -> 29.2 mm, vias 0 -> 1
- net Net-(D20-Pad1): track 0.00 -> 23.4 mm
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Other:
- board size 98.6 x 220.9 mm -> 499.1 x 299.2 mm
- board text added: "Col0"
- board text added: "Col1"
- board text added: "Col2"
- board text added: "Col3"
- board text added: "Col4"
- board text added: "MX"
- board text added: "Row0"
- board text added: "Row1"
- board text added: "Row2"
- board text added: "Row3"
- board text added: "choc"
- board text added: "cool640 designed by m.ki date 20220223 ver.1.1"
- board text added: "diode"
