File: kicad_cool640xiao/cool640xiao/cool640xiao.kicad_pcb (KiCad board)
At the start: 2 copper layers, 98.2 x 99.5 mm, 49 parts, among them J1 MJ-4PP-9, J2 MJ-4PP-9, J3 MJ-4PP-9, J4 MJ-4PP-9, SW1 SW_PUSH, SW10 SW_PUSH, SW11 SW_PUSH, SW12 SW_PUSH, SW13 SW_PUSH, SW14 SW_PUSH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

Commit message: fix
Parts:
- added D1000: D, kbd:D3_TH_SMD, F.Cu at (46.2, -6.08)
- added D1001: D, kbd:D3_TH_SMD, F.Cu at (84.4, 5.27)
- added D1002: D, kbd:D3_TH_SMD, F.Cu at (84.2, 27.0)
- added D1003: D, kbd:D3_TH_SMD, F.Cu at (84.3, 48.6)
- added D1004: D, kbd:D3_TH_SMD, F.Cu at (13.8, -10.3)
- moved D5 8.14 mm to (84.3, -5.75)
- moved D10 5.34 mm to (84.2, 16.2)
- moved D15 2.91 mm to (84.2, 37.6)
- moved D3 2.38 mm to (46.1, 4.83)
Connections:
- SW1 pad 1: col1 -> Net-(D1001-Pad1)
- SW11 pad 1: col0 -> Net-(D1000-Pad1)
- SW12 pad 1: col1 -> Net-(D1001-Pad1)
- SW13 pad 1: col3 -> Net-(D1003-Pad1)
- SW14 pad 1: col4 -> Net-(D1004-Pad1)
- SW16 pad 1: col0 -> Net-(D1000-Pad1)
- SW17 pad 1: col1 -> Net-(D1001-Pad1)
- SW18 pad 1: col2 -> Net-(D1002-Pad1)
- SW19 pad 1: col4 -> Net-(D1004-Pad1)
- SW2 pad 1: col2 -> Net-(D1002-Pad1)
- SW21 pad S1: col0 -> Net-(D1000-Pad1)
- SW22 pad S1: col1 -> Net-(D1001-Pad1)
- SW3 pad 1: col3 -> Net-(D1003-Pad1)
- SW4 pad 1: col4 -> Net-(D1004-Pad1)
- SW6 pad 1: col0 -> Net-(D1000-Pad1)
- SW7 pad 1: col2 -> Net-(D1002-Pad1)
- SW8 pad 1: col3 -> Net-(D1003-Pad1)
- SW9 pad 1: col4 -> Net-(D1004-Pad1)
Routing:
- net Net-(D1001-Pad1): track 0.00 -> 273.4 mm, vias 0 -> 3
- net Net-(D1002-Pad1): track 0.00 -> 175.2 mm
- net Net-(D1000-Pad1): track 0.00 -> 164.9 mm, vias 0 -> 2
- net col1: track 322.5 -> 176.6 mm, vias 5 -> 0
- net Net-(D1004-Pad1): track 0.00 -> 114.4 mm, vias 0 -> 1
- net Net-(D1003-Pad1): track 0.00 -> 113.8 mm, vias 0 -> 1
- net col0: track 244.9 -> 141.8 mm, vias 7 -> 0
- net col4: track 138.1 -> 65.0 mm, vias 1 -> 0
- net col2: track 230.9 -> 193.8 mm, vias 6 -> 0
- net col3: track 219.4 -> 190.8 mm, vias 0 -> 2
- net Net-(D3-Pad1): track 21.6 -> 25.1 mm
- net Net-(D5-Pad1): track 21.6 -> 18.3 mm
- net Net-(D10-Pad1): track 21.6 -> 18.3 mm
- net Net-(D15-Pad1): track 21.6 -> 19.7 mm
- net Net-(D21-Pad1): track 17.9 -> 19.5 mm
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
Commit message: fix
Parts:
- added REF**: kiritoriparts, logo:kiritoriparts, F.Cu at (153.0, 13.6)
- added REF**: kiritoriparts, logo:kiritoriparts, F.Cu at (241.3, 13.6)
- added REF**: kiritoriparts, logo:kiritoriparts, F.Cu at (241.3, -12.4)
- added REF**: kiritoriparts, logo:kiritoriparts, F.Cu at (153.0, -12.3)
Other:
- board size 98.2 x 99.5 mm -> 257.4 x 103.1 mm

Commit message: fix
Parts:
- removed REF** (x4): kiritoriparts, logo:kiritoriparts
Connections:
- D1000 pad 1: Net-(D1000-Pad1) -> col0
- D1000 pad 2: col0 -> Net-(D1000-Pad2)
- D1001 pad 1: Net-(D1001-Pad1) -> col1
- D1001 pad 2: col1 -> Net-(D1001-Pad2)
- D1002 pad 1: Net-(D1002-Pad1) -> col2
- D1002 pad 2: col2 -> Net-(D1002-Pad2)
- D1003 pad 1: Net-(D1003-Pad1) -> col3
- D1003 pad 2: col3 -> Net-(D1003-Pad2)
- SW1 pad 1: Net-(D1001-Pad1) -> Net-(D1001-Pad2)
- SW11 pad 1: Net-(D1000-Pad1) -> Net-(D1000-Pad2)
- SW12 pad 1: Net-(D1001-Pad1) -> Net-(D1001-Pad2)
- SW13 pad 1: Net-(D1003-Pad1) -> Net-(D1003-Pad2)
- SW16 pad 1: Net-(D1000-Pad1) -> Net-(D1000-Pad2)
- SW17 pad 1: Net-(D1001-Pad1) -> Net-(D1001-Pad2)
- SW18 pad 1: Net-(D1002-Pad1) -> Net-(D1002-Pad2)
- SW2 pad 1: Net-(D1002-Pad1) -> Net-(D1002-Pad2)
- SW21 pad S1: Net-(D1000-Pad1) -> Net-(D1000-Pad2)
- SW22 pad S1: Net-(D1001-Pad1) -> Net-(D1001-Pad2)
- SW3 pad 1: Net-(D1003-Pad1) -> Net-(D1003-Pad2)
- SW6 pad 1: Net-(D1000-Pad1) -> Net-(D1000-Pad2)
- SW7 pad 1: Net-(D1002-Pad1) -> Net-(D1002-Pad2)
- SW8 pad 1: Net-(D1003-Pad1) -> Net-(D1003-Pad2)
Routing:
- net Net-(D1000-Pad1): track 164.9 -> 35.4 mm, vias 2 -> 0
- net Net-(D1001-Pad1): track 273.4 -> 172.5 mm, vias 3 -> 1
- net Net-(D1003-Pad1): track 113.8 -> 57.3 mm
- net Net-(D1003-Pad2): track 0.00 -> 44.2 mm
- net Net-(D1001-Pad2): track 0.00 -> 33.5 mm
- net Net-(D1002-Pad1): track 175.2 -> 145.5 mm
- net Net-(D1000-Pad2): track 0.00 -> 24.3 mm
- net Net-(D1002-Pad2): track 0.00 -> 17.5 mm
- net col3: track 190.8 -> 182.0 mm
- net col2: track 193.8 -> 185.3 mm
- net col0: track 141.8 -> 134.7 mm
- net col1: track 176.6 -> 171.1 mm
