File: kicad_cool640xiao/cool640xiao/cool640xiao.sch (KiCad schematic (older format))
At the start: 49 parts, among them J1 MJ-4PP-9, J2 MJ-4PP-9, J3 MJ-4PP-9, J4 MJ-4PP-9, SW1 SW_PUSH, SW10 SW_PUSH, SW11 SW_PUSH, SW12 SW_PUSH, SW13 SW_PUSH, SW14 SW_PUSH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

Commit message: fix
Parts:
- added D1000, D1001, D1002, D1003, D1004: D, kbd:D3_TH_SMD, symbol Device:D
Connections:
- wire segments 77 -> 91
Other:
- moved on the sheet: J3, J4, U1

Commit message: fix
Changed lines of the file:
@@
 F 3 "~" H 5875 3525 50  0001 C CNN
 	1    5875 3525
-	-1   0    0    1
+	1    0    0    -1
 $EndComp
-Connection ~ 5725 3525
 $Comp
 L Device:D D1001
@@
 F 3 "~" H 5875 4275 50  0001 C CNN
 	1    5875 4275
-	-1   0    0    1
+	1    0    0    -1
 $EndComp
-Connection ~ 5725 4275
 $Comp
 L Device:D D1002
@@
 F 3 "~" H 5875 5025 50  0001 C CNN
 	1    5875 5025
-	-1   0    0    1
+	1    0    0    -1
 $EndComp
-Connection ~ 5725 5025
 $Comp
 L Device:D D1003
@@
 F 3 "~" H 5875 5775 50  0001 C CNN
 	1    5875 5775
-	-1   0    0    1
+	1    0    0    -1
 $EndComp
-Connection ~ 5725 5775
 $Comp
 L Device:D D1004
@@
 Wire Wire Line
 	4300 2400 4300 3125
+Connection ~ 5725 3525
+Connection ~ 5725 4275
+Connection ~ 5725 5025
+Connection ~ 5725 5775
 $EndSCHEMATC
